File: electronics/Can.kicad_sch (KiCad schematic)
At the start: 13 parts, among them J5 Conn_01x04, U6 TCAN1043xDxQ1

Commit message: Ordered this version.
Parts:
- removed C23: 1u, Capacitor_SMD:C_0402_1005Metric, symbol Device:C
- removed R17: 20k, Resistor_SMD:R_0402_1005Metric, symbol Device:R
- removed R18: 10k, Resistor_SMD:R_0402_1005Metric, symbol Device:R
- removed U6: TCAN1043xDxQ1, Package_SO:SOIC-14_3.9x8.7mm_P1.27mm, symbol Interface_CAN_LIN:TCAN1043xDxQ1
- added U6: TCAN1044A-Q1, Package_SON:VSON-8-1EP_3x3mm_P0.65mm_EP1.6x2.4mm, symbol General:TCAN1044A-Q1
- C22: renamed from C24; JLCPCB (none) -> C52923
- R18: renamed from R21; footprint Resistor_SMD:R_0603_1608Metric -> Resistor_SMD:R_0402_1005Metric; JLCPCB C22787 -> C25079
- renumbered C25 to C23, C26 to C24, J5 to J3, R19 to R16, R20 to R17
Connections:
- net 3V3: now also U6.5 (VIO)
- net CAN_RX: now also U6.4 (RXD)
- net CAN_STB: now also U6.8 (~{STB})
- net CAN_TX: now also U6.1 (TXD)
- net GND: now also J3.2 (Pin_2), U6.2 (GND)
- net VCC: now also U6.3 (VCC)
- net at D7.1 (K), R18.2: now also J3.3 (Pin_3), U6.6 (CANL); no longer J3.2 (Pin_2), J3.4 (Pin_4)
- net at D7.2 (K), R18.1: now also J3.4 (Pin_4), U6.7 (CANH); no longer J3.1 (Pin_1), J3.3 (Pin_3)
- new net VIN: J3.1 (Pin_1)
- no-connect marks 1 -> 0
Other:
- moved on the sheet: C22, D6, J3, R16, R17

Commit message: Major refactor to rev B
Connections:
- net at J3.3 (Pin_3), R18.2, U6.6 (CANL): now also D7.2 (K); no longer D7.1 (K)
- net at J3.4 (Pin_4), R18.1, U6.7 (CANH): now also D7.1 (K); no longer D7.2 (K)
Changed lines of the file:
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@@
 	(paper "A4")
 	(junction
+		(at 219.71 80.01)
+		(diameter 0)
+		(color 0 0 0 0)
+	)
+	(junction
+		(at 214.63 85.09)
+		(diameter 0)
+		(color 0 0 0 0)
+	)
+	(junction
 		(at 72.39 96.52)
 		(diameter 0)
@@
 	)
 	(junction
-		(at 219.71 85.09)
-		(diameter 0)
-		(color 0 0 0 0)
-	)
-	(junction
 		(at 162.56 25.4)
 		(diameter 0)
@@
 	)
 	(junction
-		(at 214.63 80.01)
-		(diameter 0)
-		(color 0 0 0 0)
-	)
-	(junction
 		(at 45.72 82.55)
 		(diameter 0)
@@
 	(wire
 		(pts
-			(xy 191.77 80.01) (xy 214.63 80.01)
-		)
-		(stroke
-			(width 0)
-			(type default)
-		)
-	)
-	(wire
-		(pts
 			(xy 72.39 82.55) (xy 72.39 87.63)
 		)
@@
 	(wire
 		(pts
-			(xy 224.155 88.9) (xy 224.155 83.82)
-		)
-		(stroke
-			(width 0)
-			(type default)
-		)
-	)
-	(wire
-		(pts
-			(xy 191.77 85.09) (xy 219.71 85.09)
+			(xy 224.155 88.9) (xy 224.155 85.09)
+		)
+		(stroke
+			(width 0)
+			(type default)
+		)
+	)
+	(wire
+		(pts
+			(xy 191.77 85.09) (xy 214.63 85.09)
 		)
 		(stroke
@@
 	(wire
 		(pts
-			(xy 224.155 80.01) (xy 214.63 80.01)
-		)
-		(stroke
-			(width 0)
-			(type default)
-		)
-	)
-	(wire
-		(pts
-			(xy 219.71 85.09) (xy 219.71 83.82)
+			(xy 191.77 80.01) (xy 219.71 80.01)
 		)
 		(stroke
@@
 	(wire
 		(pts
+			(xy 219.71 80.01) (xy 219.71 91.44)
+		)
+		(stroke
+			(width 0)
+			(type default)
+		)
+	)
+	(wire
+		(pts
 			(xy 179.07 100.33) (xy 179.07 107.95)
 		)
@@
 	(wire
 		(pts
-			(xy 219.71 85.09) (xy 219.71 91.44)
-		)
-		(stroke
-			(width 0)
-			(type default)
-		)
-	)
-	(wire
-		(pts
 			(xy 239.395 78.74) (xy 224.155 78.74)
 		)
@@
 	(wire
 		(pts
-			(xy 224.155 83.82) (xy 219.71 83.82)
-		)
-		(stroke
-			(width 0)
-			(type default)
-		)
-	)
-	(wire
-		(pts
 			(xy 162.56 25.4) (xy 162.56 27.94)
 		)
@@
 	(wire
 		(pts
-			(xy 214.63 80.01) (xy 214.63 91.44)
+			(xy 214.63 85.09) (xy 214.63 91.44)
 		)
 		(stroke
@@
 	(wire
 		(pts
+			(xy 219.71 80.01) (xy 224.155 80.01)
+		)
+		(stroke
+			(width 0)
+			(type default)
+		)
+	)
+	(wire
+		(pts
 			(xy 224.155 78.74) (xy 224.155 80.01)
 		)
 		(stroke
+			(width 0)
+			(type default)
+		)
+	)
+	(wire
+		(pts
+			(xy 214.63 85.09) (xy 224.155 85.09)
+		)
+		(stroke

Commit message: Refactored the design to use basic parts.
Parts:
- R16: JLCPCB C102750 -> C25741
Changed lines of the file:
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@@
 			)
 		)
-		(property "JLCPCB" "C102750"
+		(property "JLCPCB" "C25741"
 			(at 72.39 74.93 0)
 			(effects
